File: GearControl/PCB/GearControl_v2/GearControl.sch (KiCad schematic (older format))
At the start: 58 parts, among them IC1 KF50BDT-TR, J2 SWD, J6 9-6437287-8, Q1 AO3401A, Q2 2N7002, SW1 SW_SPDT, U1 MP2359DJ-LF-Z, U2 STM32F405RGT6, U4 MCP2561-E-SN, Y1 16MHz

Commit message: Add buck converter
Parts:
- IC1: symbol KF50BDT-TR:KF50BDT-TR -> GearControl-rescue:KF50BDT-TR-KF50BDT-TR
- J6: symbol 9-6437287-8:9-6437287-8 -> GearControl-rescue:9-6437287-8-9-6437287-8
Changed lines of the file:
@@
 EESchema Schematic File Version 4
-LIBS:GearControl-cache
-EELAYER 29 0
+EELAYER 30 0
 EELAYER END
 $Descr A4 11693 8268
@@
 	750  900  750  1175
 $Comp
-L 9-6437287-8:9-6437287-8 J6
+L GearControl-rescue:9-6437287-8-9-6437287-8 J6
 U 1 1 6180B151
 P 10225 5100
@@
 NoConn ~ 3075 6575
 $Comp
-L KF50BDT-TR:KF50BDT-TR IC1
+L GearControl-rescue:KF50BDT-TR-KF50BDT-TR IC1
 U 1 1 61945E33
 P 6375 2725
