File: Dashboard/PCB/Dashboard.sch (KiCad schematic (older format))
At the start: 92 parts, among them J1 Display, J2 Conn_01x26_Female, J3 LED, J7 PROGRAMMER, P1 USB_C_Plug, SW1 SW_SPST, U1 STM32F767ZIT6, U10 24LC01, U3 MP2359DJ-LF-Z, U4 AS4C1M16S-6TCN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

Commit message: Add LED Driver
Parts:
- added C32: 100nF, Capacitor_SMD:C_0805_2012Metric, symbol Device:C
- added Q1: Q_NMOS_GDS, Package_TO_SOT_SMD:SOT-89-3_Handsoldering, symbol Device:Q_NMOS_GDS
- added R13, R9: R, Resistor_SMD:R_0805_2012Metric, symbol Device:R
- added R20: 1R, Resistor_SMD:R_0805_2012Metric, symbol Device:R
Connections:
- net +12L: now also Q1.2 (D)
- net +5V: no longer J1.2 (Pin_2)
- net GND: now also C32.2, R20.2; no longer J1.1 (Pin_1), R16.2
- net LED_CURRENT_SENSE: now reaches U1.27 (PC1(TRACED0,DFSDM1_DATIN0,SAI2_MOSI/I2S2_SD,SAI1_SD_A,DFSDM1_CKIN4,ETH_MDC,MDIOS_MDC,ADC1_IN11,ADC2_IN11,ADC3_IN11,RTC_TAMP3))
- net LED_CURRENT_SENSE: now also C32.1, R9.2
- net LED_PWM: now reaches U1.81 (PD12(TIM4_CH1,LPTIM1_IN1,I2C4_SCL,USART3_RTS,QUADSPI_BK1_IO1,SAI2_FS_A,FMC_A17/FMC_ALE))
- net LED_PWM: now also R13.2
- new net: Q1.1 (G), R13.1
- new net DISPLAY_LED+: J1.2 (Pin_2), Q1.3 (S)
- new net DISPLAY_LED-: J1.1 (Pin_1), R20.1, R9.1
- no-connect marks 41 -> 39
Other:
- note added: "Made in China\n"
- moved on the sheet: C1, C10, C11, C12, C13, C14, C15, C17, C18, C2, C3, C31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
