File: Dashboard/PCB/Dashboard.sch (KiCad schematic (older format))
At the start: 91 parts, among them J1 Display, J2 Conn_01x26_Female, J3 LED, J7 PROGRAMMER, SW1 SW_SPST, U1 STM32F767ZIT6, U10 24LC01, U3 MP2359DJ-LF-Z, U4 AS4C1M16S-6TCN, U5 AT25SF128A-SHB-T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

Commit message: PCB v1.0 (#21)
* Add usb C to board

* Add reset and pd pin to esp

* Switch footprints of converter

* Add LED Driver

* Add text to pcb
Parts:
- removed R19: 10k, Resistor_SMD:R_0805_2012Metric, symbol Device:R
- added C32: 100nF, Capacitor_SMD:C_0805_2012Metric, symbol Device:C
- added D6, D7: D_Schottky, Diode_SMD:D_0805_2012Metric_Pad1.15x1.40mm_HandSolder, symbol Device:D_Schottky
- added P1: USB_C_Plug, Connector_USB:USB_C_Receptacle_Amphenol_12401548E4-2A, symbol Connector:USB_C_Plug
- added Q1: Q_NMOS_GDS, Package_TO_SOT_SMD:SOT-89-3_Handsoldering, symbol Device:Q_NMOS_GDS
- added R13, R9: R, Resistor_SMD:R_0805_2012Metric, symbol Device:R
- R20: value 10k -> 1R
- U3: footprint Package_SO:SOIC-8-1EP_3.9x4.9mm_P1.27mm_EP2.29x3mm -> SOT-583:SOTFL50P160X60-8N
- U6: footprint SOT-583:SOTFL50P160X60-8N -> Package_SO:SOIC-8-1EP_3.9x4.9mm_P1.27mm_EP2.29x3mm
Connections:
- net +12L: now also D6.1 (K), D7.1 (K), Q1.2 (D)
- net +5V: no longer J1.2 (Pin_2)
- net GND: now also R20.2, C32.2, P1.A1 (GND), P1.A12 (GND), P1.B1 (GND), P1.B12 (GND), P1.S1 (SHIELD); no longer J1.1 (Pin_1), J7.5 (Pin_5), R16.2
- net USB_OTG_DM: now reaches U1.75 (PB14(TIM1_CH2N,TIM8_CH2N,USART1_TX,SPI2_MISO,DFSDM1_DATIN2,USART3_RTS,UART4_RTS,TIM12_CH1,SDMMC2_D0,OTG_HS_DM))
- net USB_OTG_DM: now also P1.A7 (D-)
- net USB_OTG_DP: now reaches U1.76 (PB15(RTC_REFIN,TIM1_CH3N,TIM8_CH3N,USART1_RX,SPI2_MOSI/I2S2_SD,DFSDM1_CKIN2,UART4_CTS,TIM12_CH2,SDMMC2_D1,OTG_HS_DP))
- net USB_OTG_DP: now also P1.A6 (D+)
- net ESP_RESET: now reaches U1.111 (PC10(DFSDM1_CKIN5,SPI3_SCK/I2S3_CK,USART3_TX,UART4_TX,QUADSPI_BK1_IO1,SDMMC1_D2,DCMI_D8,LCD_R2))
- net ESP_RESET: now also U9.1 (RST)
- net ESP_EN: now reaches U1.112 (PC11(DFSDM1_DATIN5,SPI3_MISO,USART3_RX,UART4_RX,QUADSPI_BK2_NCS,SDMMC1_D3,DCMI_D4))
- net ESP_EN: now also U9.3 (EN)
- net LED_CURRENT_SENSE: now reaches U1.27 (PC1(TRACED0,DFSDM1_DATIN0,SAI2_MOSI/I2S2_SD,SAI1_SD_A,DFSDM1_CKIN4,ETH_MDC,MDIOS_MDC,ADC1_IN11,ADC2_IN11,ADC3_IN11,RTC_TAMP3))
- net LED_CURRENT_SENSE: now also C32.1, R9.2
- net LED_PWM: now reaches U1.81 (PD12(TIM4_CH1,LPTIM1_IN1,I2C4_SCL,USART3_RTS,QUADSPI_BK1_IO1,SAI2_FS_A,FMC_A17/FMC_ALE))
- net LED_PWM: now also R13.2
- net DISPLAY_LED-: now reaches R20.1
- net DISPLAY_LED-: now also J1.1 (Pin_1), R9.1
- new net: D6.2 (A), P1.A4 (VBUS), P1.A9 (VBUS), P1.B4 (VBUS), P1.B9 (VBUS)
- new net: D7.2 (A), J7.5 (Pin_5)
- new net: Q1.1 (G), R13.1
- new net DISPLAY_LED+: J1.2 (Pin_2), Q1.3 (S)
- no-connect marks 45 -> 39
Other:
- note added: "Made in China\n"
- moved on the sheet: C1, C10, C11, C12, C13, C14, C15, C17, C18, C2, C3, C31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
