File: Telemetry/PCB/back/_autosave-telemetria tyl.sch (KiCad schematic (older format))
At the start: 61 parts, among them J1 Conn_01x26_Male, J2 Conn_02x05_Odd_Even, U1 STM32F405RGTx, U2 MCP2561-E-SN, Y1 Crystal_GND24_Small

Commit message: final scheme & 60%pcb
Parts:
- PS1, PS2: footprint SOT-583:SOTFL50P160X60-8N -> Package_SO:SOIC-8-1EP_3.9x4.9mm_P1.27mm_EP2.29x3mm_ThermalVias
Changed lines of the file:
@@
 F 0 "PS2" H 9600 3265 50  0000 C CNN
 F 1 "MP2359DT-LF-P" H 9600 3174 50  0000 C CNN
-F 2 "SOT-583:SOTFL50P160X60-8N" H 9950 3100 50  0001 L CNN
+F 2 "Package_SO:SOIC-8-1EP_3.9x4.9mm_P1.27mm_EP2.29x3mm_ThermalVias" H 9950 3100 50  0001 L CNN
 F 3 "https://ms.componentsearchengine.com/Datasheets/2/MP2359DT-LF-P.pdf" H 9950 3000 50  0001 L CNN
 F 4 "MONOLITHIC POWER SYSTEMS (MPS) - MP2359DT-LF-P - DC-DC Switching Buck (Step Down) Regulator, 4.5V-24V in, 810mV to 15V out, 1.2A, 1.4MHz, SOT-23-6" H 9950 2900 50  0001 L CNN "Description"
@@
 F 0 "PS1" H 9100 4665 50  0000 C CNN
 F 1 "MP2359DT-LF-P" H 9100 4574 50  0000 C CNN
-F 2 "SOT-583:SOTFL50P160X60-8N" H 9450 4500 50  0001 L CNN
+F 2 "Package_SO:SOIC-8-1EP_3.9x4.9mm_P1.27mm_EP2.29x3mm_ThermalVias" H 9450 4500 50  0001 L CNN
 F 3 "https://ms.componentsearchengine.com/Datasheets/2/MP2359DT-LF-P.pdf" H 9450 4400 50  0001 L CNN
 F 4 "MONOLITHIC POWER SYSTEMS (MPS) - MP2359DT-LF-P - DC-DC Switching Buck (Step Down) Regulator, 4.5V-24V in, 810mV to 15V out, 1.2A, 1.4MHz, SOT-23-6" H 9450 4300 50  0001 L CNN "Description"
@@
 	7600 4400 7600 4550
 $Comp
-L power:+3.3V #PWR0116
-U 1 1 627F0F17
-P 9000 3950
-F 0 "#PWR0116" H 9000 3800 50  0001 C CNN
-F 1 "+3.3V" H 9015 4123 50  0000 C CNN
-F 2 "" H 9000 3950 50  0001 C CNN
-F 3 "" H 9000 3950 50  0001 C CNN
-	1    9000 3950
-	1    0    0    -1
-$EndComp
-$Comp
 L power:GND #PWR0117
 U 1 1 627F0F1D
@@
 	10950 3450 11100 3450
 Connection ~ 11100 3150
+$Comp
+L power:+5V #PWR0116
+U 1 1 629909F8
+P 9000 3950
+F 0 "#PWR0116" H 9000 3800 50  0001 C CNN
+F 1 "+5V" H 9015 4123 50  0000 C CNN
+F 2 "" H 9000 3950 50  0001 C CNN
+F 3 "" H 9000 3950 50  0001 C CNN
+	1    9000 3950
+	1    0    0    -1
+$EndComp
 $EndSCHEMATC
