File: Telemetry/PCB/back/telemetria tyl.kicad_pcb (KiCad board)
At the start: 2 copper layers, 60 parts, among them J1 Conn_01x26_Male, U1 STM32F405RGTx, U2 MCP2561-E-SN, Y1 Crystal_GND24_Small

Commit message: pre_finnal
Parts:
- added 2channel_pot1: MAX5478EUD+T, SamacSys_Parts:SOP65P640X110-14N, F.Cu at (53.3, 66.6)
- added BJT1: BC846BW,115, SamacSys_Parts:SOT65P210X110-3N, F.Cu at (28.3, 74.9)
- added C10: C, Capacitor_SMD:C_0805_2012Metric_Pad1.18x1.45mm_HandSolder, F.Cu at (43.2, 35.6)
- added C11: C, Capacitor_SMD:C_0805_2012Metric_Pad1.18x1.45mm_HandSolder, F.Cu at (41.9, 57.1)
- added C21: C, Capacitor_SMD:C_0805_2012Metric_Pad1.18x1.45mm_HandSolder, F.Cu at (41.9, 54.0)
- added C22: C, Capacitor_SMD:C_0805_2012Metric_Pad1.18x1.45mm_HandSolder, F.Cu at (38.1, 35.6)
- added C9: 0.1uF, Capacitor_SMD:C_0805_2012Metric_Pad1.18x1.45mm_HandSolder, F.Cu at (59.7, 65.8)
- added IC1: LM741CN_NOPB, DIP794W53P254L959H508Q8N, F.Cu at (47.0, 77.5)
- added IC2: LM741CN_NOPB, DIP794W53P254L959H508Q8N, F.Cu at (41.9, 43.2)
- added IC3: LM741CN_NOPB, DIP794W53P254L959H508Q8N, F.Cu at (43.2, 66.0)
- added J2: Conn_02x05_Odd_Even, Connector_PinHeader_2.54mm:PinHeader_2x05_P2.54mm_Vertical, F.Cu at (67.3, 26.7)
- added Mini_DIN_IN1: 5749268-1, SamacSys_Parts:57492681, F.Cu at (30.5, 44.5)
- added Mini_DIN_OUT1: 5750071-1, SamacSys_Parts:57500711, F.Cu at (30.5, 64.8)
- added R10: R, Resistor_SMD:R_0805_2012Metric_Pad1.20x1.40mm_HandSolder, F.Cu at (45.7, 35.6)
- added R14: R, Resistor_SMD:R_0805_2012Metric_Pad1.20x1.40mm_HandSolder, F.Cu at (49.5, 40.6)
- added R15: R, Resistor_SMD:R_0805_2012Metric_Pad1.20x1.40mm_HandSolder, F.Cu at (40.6, 50.8)
- added R16: R, Resistor_SMD:R_0805_2012Metric_Pad1.20x1.40mm_HandSolder, F.Cu at (43.2, 50.8)
- added R17: R, Resistor_SMD:R_0805_2012Metric_Pad1.20x1.40mm_HandSolder, F.Cu at (38.1, 55.9)
- added R18: R, Resistor_SMD:R_0805_2012Metric_Pad1.20x1.40mm_HandSolder, F.Cu at (39.6, 73.7)
- added R19: R?, Resistor_SMD:R_0805_2012Metric_Pad1.20x1.40mm_HandSolder, F.Cu at (54.3, 71.1)
- added R9: 1M, Resistor_SMD:R_0805_2012Metric_Pad1.20x1.40mm_HandSolder, F.Cu at (40.6, 35.6)
- PS1, PS2: footprint Package_SO:SOIC-8-1EP_3.9x4.9mm_P1.27mm_EP2.29x3mm_ThermalVias -> SamacSys_Parts:SOT95P280X145-6N
- moved D5 17.3 mm to (69.8, 69.8)
- moved R13 17.3 mm to (69.8, 72.4)
- moved D3 10.1 mm to (75.4, 69.8), turned to 180 degrees
- moved R12 10.0 mm to (75.5, 72.4), turned to 180 degrees
- moved H1 6.10 mm to (35.6, 78.7)
- moved H2 6.10 mm to (35.6, 25.7)
- moved C8 1.83 mm to (50.8, 36.8), turned to 0 degrees
- moved C7 1.69 mm to (50.8, 34.3), turned to 0 degrees
- moved 10k1 1.27 mm to (67.1, 39.9)
- moved H4 0.76 mm to (92.5, 25.4)
Routing:
- net GND: track 231.4 -> 326.4 mm, vias 15 -> 16
- net GND_MIC&ANC: track 0.00 -> 88.8 mm, vias 0 -> 2
- net +5V: track 48.7 -> 118.4 mm
- net SWDIO: track 0.00 -> 62.9 mm, vias 0 -> 3
- net NRST: track 0.00 -> 53.8 mm, vias 0 -> 1
- net SWO: track 0.00 -> 43.8 mm, vias 0 -> 2
- net V_OUT: track 0.00 -> 36.9 mm
- net SWCLK: track 0.00 -> 35.6 mm, vias 0 -> 1
- net V_MIC: track 0.00 -> 34.0 mm, vias 0 -> 1
- net GND_SPK: track 0.00 -> 33.8 mm
- net 12C2_SDA: track 29.8 -> 57.3 mm, vias 2 -> 6
- net Net-(2channel_pot1-Pad1): track 0.00 -> 27.0 mm
- net Net-(IC2-Pad2): track 0.00 -> 22.0 mm
- net Net-(2channel_pot1-Pad2): track 0.00 -> 21.4 mm
- net TX_DATA: track 0.00 -> 21.2 mm
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Other:
- board text added: "Janicki & Szamocki"
- board text added: "Telemetry back"

Commit message: pre_finnal
Connections:
- C13 pad 1: Net-(C13-Pad1) -> +3V3
- C14 pad 1: Net-(C13-Pad1) -> +3V3
- C15 pad 1: Net-(C13-Pad1) -> +3V3
- C16 pad 1: Net-(C13-Pad1) -> +3V3
- C17 pad 1: Net-(C13-Pad1) -> +3V3
- C18 pad 1: Net-(C13-Pad1) -> +3V3
- C19 pad 1: Net-(C13-Pad1) -> +3V3
- C20 pad 1: Net-(C13-Pad1) -> +3V3
Routing:
- net Net-(C13-Pad1): track 16.9 -> 0.00 mm
- net +3V3: track 209.3 -> 226.2 mm

Commit message: telemetry_back_finnal
Parts:
- added G***: LOGO, SamacSys_Parts:logo, F.Cu at (106.7, 80.0)
- added G***: LOGO, SamacSys_Parts:logo, F.Cu at (25.4, 25.4)
- added IC4: NCX2200GW,125, SamacSys_Parts:NCX2200GW, B.Cu at (73.7, 78.7)
- added Q1: PMF250XNEX, SamacSys_Parts:PMF250XNEX, B.Cu at (77.5, 78.7)
- added R20: 3.3k, Resistor_SMD:R_0805_2012Metric_Pad1.20x1.40mm_HandSolder, B.Cu at (73.8, 82.8)
- added RV1: R_POT, Potentiometer_THT:Potentiometer_Alps_RK09L_Single_Vertical, F.Cu at (58.4, 74.9)
- BJT1: moved to B.Cu
- moved BJT1 18.8 mm to (43.2, 63.5), turned to 180 degrees
- moved 0.33k1 0.20 mm to (64.5, 60.9)
- moved 0.33k2 0.20 mm to (66.8, 60.9)
Connections:
- net ADC1_IN0 renamed ADC1_IN0_AMORKI
- net ADC2_IN1 renamed ADC2_IN1_AMORKI
- BJT1 pad 1: 3.3V -> PTT
- J1 pad 24: Net-(J1-Pad24) -> BREAK_PRESSURE_0
- J1 pad 25: Net-(J1-Pad25) -> BREAK_PRESSURE_ADC
- J1 pad 26: Net-(J1-Pad26) -> LED_GND
- U1 pad 17: Net-(U1-Pad17) -> BREAK_PRESSURE_0
- U1 pad 20: Net-(U1-Pad20) -> BREAK_PRESSURE_ADC
- U1 pad 8: Net-(U1-Pad8) -> PTT
Routing:
- net GND: track 326.4 -> 444.3 mm
- net BREAK_PRESSURE_0: track 0.00 -> 46.4 mm, vias 0 -> 3
- net BREAK_PRESSURE_ADC: track 0.00 -> 29.3 mm, vias 0 -> 2
- net PTT: track 0.00 -> 23.5 mm, vias 0 -> 1
- net LED_GND: track 0.00 -> 21.2 mm, vias 0 -> 1
- net GND_SPK: track 33.8 -> 55.0 mm
- net +5V: track 118.4 -> 134.2 mm, vias 4 -> 5
- net Net-(IC4-Pad4): track 0.00 -> 13.3 mm
- net Net-(Q1-Pad1): track 0.00 -> 9.28 mm, vias 0 -> 2
- net GND_MIC&ANC: track 88.8 -> 94.3 mm
- net Net-(IC4-Pad1): track 0.00 -> 3.93 mm
- net +3V3: track 226.2 -> 227.3 mm
Other:
- board text added: "Telemetry back v 1.0 Janicki & Szamocki"
- board text removed: "Janicki & Szamocki"
- board text removed: "Telemetry back"

Commit message: Telemetry_back_finnal
Parts:
- added R21: 4.7k, Resistor_SMD:R_0805_2012Metric_Pad1.20x1.40mm_HandSolder, B.Cu at (50.8, 61.0)
- added R22: 1k, Resistor_SMD:R_0805_2012Metric_Pad1.20x1.40mm_HandSolder, B.Cu at (53.3, 61.0)
Connections:
- BJT1 pad 1: PTT -> Net-(BJT1-Pad1)
- BJT1 pad 3: GND_MIC&ANC -> Net-(BJT1-Pad3)
Routing:
- net Net-(BJT1-Pad3): track 0.00 -> 15.6 mm
- net Net-(BJT1-Pad1): track 0.00 -> 7.42 mm
- net PTT: track 23.5 -> 17.9 mm
- net GND_MIC&ANC: track 94.3 -> 97.3 mm
Other:
- board text added: "Telemetry back v 1.0 Szamocki & Janicki"
