File: Telemetry/PCB/back/telemetria tyl.sch (KiCad schematic (older format))
At the start: 61 parts, among them J1 Conn_01x26_Male, J2 Conn_02x05_Odd_Even, U1 STM32F405RGTx, U2 MCP2561-E-SN, Y1 Crystal_GND24_Small

Commit message: pre_finnal
Parts:
- added 2channel_pot1: MAX5478EUD+T, SamacSys_Parts:SOP65P640X110-14N, symbol MAX5478EUD+T:MAX5478EUD+T
- added BJT1: BC846BW,115, SamacSys_Parts:SOT65P210X110-3N, symbol BC846BW:BC846BW
- added C10, C11, C21, C22: C, Capacitor_SMD:C_0805_2012Metric_Pad1.18x1.45mm_HandSolder, symbol Device:C
- added C9: 0.1uF, Capacitor_SMD:C_0805_2012Metric_Pad1.18x1.45mm_HandSolder, symbol Device:C
- added IC1, IC2, IC3: LM741CN_NOPB, DIP794W53P254L959H508Q8N, symbol LM741CN_NOPB:LM741CN_NOPB
- added Mini_DIN_IN1: 5749268-1, SamacSys_Parts:57492681, symbol 5749268-1:5749268-1
- added Mini_DIN_OUT1: 5750071-1, SamacSys_Parts:57500711, symbol 5750071-1:5750071-1
- added R10, R14, R15, R16, R17, R18: R, Resistor_SMD:R_0805_2012Metric_Pad1.20x1.40mm_HandSolder, symbol Device:R
- added R19: R?, Resistor_SMD:R_0805_2012Metric_Pad1.20x1.40mm_HandSolder, symbol Device:R
- added R9: 1M, Resistor_SMD:R_0805_2012Metric_Pad1.20x1.40mm_HandSolder, symbol Device:R
- PS1, PS2: footprint Package_SO:SOIC-8-1EP_3.9x4.9mm_P1.27mm_EP2.29x3mm_ThermalVias -> SamacSys_Parts:SOT95P280X145-6N; symbol MP2359DT-LF-P:MP2359DT-LF-P -> telemetria-tyl-rescue:MP2359DT-LF-P-MP2359DT-LF-P
Connections:
- net labels added: 3.3V, GND_MIC&ANC, GND_SPK, SPK+, TX_DATA, V_ANC, V_MIC, V_OUT
- wire segments 163 -> 210
- no-connect marks 0 -> 25
Other:
- note added: "DIN_IN\n"
- note added: "DIN_OUT\n"
- note added: "PUSH TO TALK //SPRAWDZIC W PROTO\n"
- moved on the sheet: 0.33k1, 0.33k2, 10k1, 10nF1, 1k1, 1k2, 1uF1, 2.2uF1, 2.2uF2, 39nH1, C1, C12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

Commit message: telemetry_back_finnal
Parts:
- added IC4: NCX2200GW,125, SamacSys_Parts:NCX2200GW, symbol NCX2200GW_125:NCX2200GW,125
- added Q1: PMF250XNEX, SamacSys_Parts:PMF250XNEX, symbol PMF250XNEX:PMF250XNEX
- added R20: 3.3k, Resistor_SMD:R_0805_2012Metric_Pad1.20x1.40mm_HandSolder, symbol Device:R
- added RV1: R_POT, Potentiometer_THT:Potentiometer_Alps_RK09L_Single_Vertical, symbol Device:R_POT
Connections:
- net labels added: ADC1_IN0_AMORKI, ADC2_IN1_AMORKI, BREAK_PRESSURE_0, BREAK_PRESSURE_ADC, LED_GND, PTT
- net labels removed: 3.3V, ADC1_IN0, ADC2_IN1
- wire segments 210 -> 214
- no-connect marks 25 -> 26
Other:
- moved on the sheet: 0.33k1, 0.33k2, 1k1, 1k2

Commit message: Telemetry_back_finnal
Parts:
- added R21: 4.7k, Resistor_SMD:R_0805_2012Metric_Pad1.20x1.40mm_HandSolder, symbol Device:R
- added R22: 1k, Resistor_SMD:R_0805_2012Metric_Pad1.20x1.40mm_HandSolder, symbol Device:R
Connections:
- net GND_MIC&ANC: now also R22.1; no longer BJT1.3 (C)
- net PTT: now also R21.2; no longer BJT1.1 (B)
- new net: BJT1.1 (B), R21.1
- new net: BJT1.3 (C), R22.2
Changed lines of the file:
@@
 NoConn ~ 5050 7400
 NoConn ~ 3700 5750
-Text GLabel 3750 7050 2    50   Input ~ 0
+Text GLabel 4050 7050 2    50   Input ~ 0
 GND_MIC&ANC
 Text GLabel 2950 7150 0    50   Input ~ 0
@@
 Text GLabel 4400 5900 0    50   Input ~ 0
 SPK+
-$Comp
-L BC846BW:BC846BW BJT1
-U 1 1 62596133
-P 2950 7050
-F 0 "BJT1" H 3350 7315 50  0000 C CNN
-F 1 "BC846BW,115" H 3350 7224 50  0000 C CNN
-F 2 "SamacSys_Parts:SOT65P210X110-3N" H 3600 7150 50  0001 L CNN
-F 3 "http://www.nxp.com/documents/data_sheet/BC846_SER.pdf" H 3600 7050 50  0001 L CNN
-F 4 "Bipolar Transistors - BJT TRANS GP TAPE-7" H 3600 6950 50  0001 L CNN "Description"
-F 5 "1.1" H 3600 6850 50  0001 L CNN "Height"
-F 6 "771-BC846BW-T/R" H 3600 6750 50  0001 L CNN "Mouser Part Number"
-F 7 "https://www.mouser.co.uk/ProductDetail/Nexperia/BC846BW115?qs=me8TqzrmIYXeHaJTKQ9DIQ%3D%3D" H 3600 6650 50  0001 L CNN "Mouser Price/Stock"
-F 8 "Nexperia" H 3600 6550 50  0001 L CNN "Manufacturer_Name"
-F 9 "BC846BW,115" H 3600 6450 50  0001 L CNN "Manufacturer_Part_Number"
-	1    2950 7050
-	1    0    0    -1
-$EndComp
 Text GLabel 4400 5800 0    50   Input ~ 0
 GND_MIC&ANC
@@
 Text GLabel 1300 2850 0    50   Input ~ 0
 PTT
-Text GLabel 2950 7050 0    50   Input ~ 0
+$Comp
+L Device:R R22
+U 1 1 629D953B
+P 3900 7050
+F 0 "R22" V 3693 7050 50  0000 C CNN
+F 1 "1k" V 3784 7050 50  0000 C CNN
+F 2 "Resistor_SMD:R_0805_2012Metric_Pad1.20x1.40mm_HandSolder" V 3830 7050 50  0001 C CNN
+F 3 "~" H 3900 7050 50  0001 C CNN
+	1    3900 7050
+	0    1    1    0
+$EndComp
+$Comp
+L Device:R R21
+U 1 1 629DA4E2
+P 2800 7050
+F 0 "R21" V 2593 7050 50  0000 C CNN
+F 1 "4.7k" V 2684 7050 50  0000 C CNN
+F 2 "Resistor_SMD:R_0805_2012Metric_Pad1.20x1.40mm_HandSolder" V 2730 7050 50  0001 C CNN
+F 3 "~" H 2800 7050 50  0001 C CNN
+	1    2800 7050
+	0    1    1    0
+$EndComp
+Text GLabel 2650 7050 0    50   Input ~ 0
 PTT
+$Comp
+L BC846BW:BC846BW BJT1
+U 1 1 62596133
+P 2950 7050
+F 0 "BJT1" H 3350 7315 50  0000 C CNN
+F 1 "BC846BW,115" H 3350 7224 50  0000 C CNN
+F 2 "SamacSys_Parts:SOT65P210X110-3N" H 3600 7150 50  0001 L CNN
+F 3 "http://www.nxp.com/documents/data_sheet/BC846_SER.pdf" H 3600 7050 50  0001 L CNN
+F 4 "Bipolar Transistors - BJT TRANS GP TAPE-7" H 3600 6950 50  0001 L CNN "Description"
+F 5 "1.1" H 3600 6850 50  0001 L CNN "Height"
+F 6 "771-BC846BW-T/R" H 3600 6750 50  0001 L CNN "Mouser Part Number"
+F 7 "https://www.mouser.co.uk/ProductDetail/Nexperia/BC846BW115?qs=me8TqzrmIYXeHaJTKQ9DIQ%3D%3D" H 3600 6650 50  0001 L CNN "Mouser Price/Stock"
+F 8 "Nexperia" H 3600 6550 50  0001 L CNN "Manufacturer_Name"
+F 9 "BC846BW,115" H 3600 6450 50  0001 L CNN "Manufacturer_Part_Number"
+	1    2950 7050
+	1    0    0    -1
+$EndComp
 $EndSCHEMATC

Commit message: finnal
Parts:
- removed JP1: Jumper_3_Bridged12, Jumper:SolderJumper-3_P1.3mm_Open_RoundedPad1.0x1.5mm, symbol Jumper:Jumper_3_Bridged12
- removed JP2: Jumper, Jumper:SolderJumper-2_P1.3mm_Open_Pad1.0x1.5mm, symbol Device:Jumper
- removed Q1: PMF250XNEX, SamacSys_Parts:PMF250XNEX, symbol PMF250XNEX:PMF250XNEX
- added C23: ?, Capacitor_SMD:C_0805_2012Metric_Pad1.18x1.45mm_HandSolder, symbol Device:C
- added C24: 10uF, Capacitor_SMD:C_0805_2012Metric_Pad1.18x1.45mm_HandSolder, symbol Device:C
- added Q1: PMV280ENEAR, SamacSys_Parts:PMV280ENEAR, symbol PMV280ENEAR:PMV280ENEAR
- added R23: R, Resistor_SMD:R_0805_2012Metric_Pad1.20x1.40mm_HandSolder, symbol Device:R
- R4: value R -> 120
Connections:
- net +3V3: now also R23.2
- net +5V: now also U2.3 (VDD)
- net CAN_H1: now also R4.1
- net GND: now also Q1.2
- net GND_MIC&ANC: now also C23.1, C24.1
- net LED_GND: now also Q1.3
- net V_ANC: now also C23.2, C24.2, R23.1
- net at R20.2: now also Q1.1
Other:
- note added: "PUSH TO TALK \n"
- note removed: "PUSH TO TALK //SPRAWDZIC W PROTO\n"
- moved on the sheet: 2channel_pot1, BJT1, C10, C11, C21, C22, C9, IC1, IC2, IC3, IC4, Mini_DIN_IN1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
