File: Telemetry/PCB/back/telemetria tyl.sch (KiCad schematic (older format))
At the start: 88 parts, among them IC1 LM741CN_NOPB, IC2 LM741CN_NOPB, IC3 LM741CN_NOPB, IC4 NCX2200GW,125, J1 Conn_01x26_Male, J2 Conn_02x05_Odd_Even, Q1 PMV280ENEAR, U1 STM32F405RGTx, U2 MCP2561-E-SN, Y1 16Mhz

Commit message: Telemetry_back_v1.1
Parts:
- D1, D3, D5: value LED_5V -> LED_3.2V
- R12, R13: value 260 -> 360
- R7: value 510 -> 820
- R8: value 1k7 -> 2k7
Changed lines of the file:
@@
 P 10250 1750
 F 0 "R13" V 10043 1750 50  0000 C CNN
-F 1 "260" V 10134 1750 50  0000 C CNN
+F 1 "360" V 10134 1750 50  0000 C CNN
 F 2 "Resistor_SMD:R_0805_2012Metric_Pad1.20x1.40mm_HandSolder" V 10180 1750 50  0001 C CNN
 F 3 "~" H 10250 1750 50  0001 C CNN
@@
 P 9000 1450
 F 0 "D1" V 9039 1332 50  0000 R CNN
-F 1 "LED_5V" V 8948 1332 50  0000 R CNN
+F 1 "LED_3.2V" V 8948 1332 50  0000 R CNN
 F 2 "Diode_SMD:D_0805_2012Metric_Pad1.15x1.40mm_HandSolder" H 9000 1450 50  0001 C CNN
 F 3 "~" H 9000 1450 50  0001 C CNN
@@
 P 9650 1500
 F 0 "D3" V 9689 1382 50  0000 R CNN
-F 1 "LED_5V" V 9598 1382 50  0000 R CNN
+F 1 "LED_3.2V" V 9598 1382 50  0000 R CNN
 F 2 "Diode_SMD:D_0805_2012Metric_Pad1.15x1.40mm_HandSolder" H 9650 1500 50  0001 C CNN
 F 3 "~" H 9650 1500 50  0001 C CNN
@@
 P 10250 1450
 F 0 "D5" V 10289 1332 50  0000 R CNN
-F 1 "LED_5V" V 10198 1332 50  0000 R CNN
+F 1 "LED_3.2V" V 10198 1332 50  0000 R CNN
 F 2 "Diode_SMD:D_0805_2012Metric_Pad1.15x1.40mm_HandSolder" H 10250 1450 50  0001 C CNN
 F 3 "~" H 10250 1450 50  0001 C CNN
@@
 P 8800 2650
 F 0 "R7" V 8593 2650 50  0000 C CNN
-F 1 "510" V 8684 2650 50  0000 C CNN
+F 1 "820" V 8684 2650 50  0000 C CNN
 F 2 "Resistor_SMD:R_0805_2012Metric_Pad1.20x1.40mm_HandSolder" V 8730 2650 50  0001 C CNN
 F 3 "~" H 8800 2650 50  0001 C CNN
@@
 P 9100 2650
 F 0 "R8" V 8893 2650 50  0000 C CNN
-F 1 "1k7" V 8984 2650 50  0000 C CNN
+F 1 "2k7" V 8984 2650 50  0000 C CNN
 F 2 "Resistor_SMD:R_0805_2012Metric_Pad1.20x1.40mm_HandSolder" V 9030 2650 50  0001 C CNN
 F 3 "~" H 9100 2650 50  0001 C CNN
@@
 	7250 4350 7400 4350
 Wire Wire Line
-	7250 4150 7250 4350
+	7200 5300 7200 5500
 Wire Wire Line
 	6800 4150 7250 4150
@@
 P 9650 1800
 F 0 "R12" V 9443 1800 50  0000 C CNN
-F 1 "260" V 9534 1800 50  0000 C CNN
+F 1 "360" V 9534 1800 50  0000 C CNN
 F 2 "Resistor_SMD:R_0805_2012Metric_Pad1.20x1.40mm_HandSolder" V 9580 1800 50  0001 C CNN
 F 3 "~" H 9650 1800 50  0001 C CNN
@@
 	1    0    0    -1
 $EndComp
+Wire Wire Line
+	7250 4150 7250 4350
 $EndSCHEMATC
