File: Telemetry/PCB/back/telemetria tyl.sch (KiCad schematic (older format))
At the start: 23 parts

Commit message: final scheme & 60%pcb
Parts:
- removed C?: 100nF, symbol Device:C
- removed C? (x2): 10uF, symbol Device:C
- removed D?: D_Schottky, symbol Device:D_Schottky
- removed D?: 1N4148, Diode_THT:D_DO-35_SOD27_P7.62mm_Horizontal, symbol Diode:1N4148
- removed IC?: MP2333HGTL, SOTFL50P160X60-8N, symbol MP2333HGTL:MP2333HGTL
- removed L?: 10uH, symbol Device:L
- removed PS?: MP2359DT-LF-P, SOT95P280X145-6N, symbol MP2359DT-LF-P:MP2359DT-LF-P
- removed R? (x3): R, symbol Device:R
- removed R?: 100k, symbol Device:R
- added 0.33k1, 0.33k2, 10k1, 1k1, 1k2, R11, R12, R13, R5, R6, R7, R8: R, Resistor_SMD:R_0805_2012Metric_Pad1.20x1.40mm_HandSolder, symbol Device:R
- added 10nF1, 1uF1: C1, Capacitor_SMD:C_0805_2012Metric_Pad1.18x1.45mm_HandSolder, symbol Device:C
- added 2.2uF1, 2.2uF2: C_Small, Capacitor_SMD:C_0805_2012Metric_Pad1.18x1.45mm_HandSolder, symbol Device:C_Small
- added 39nH1: 39nH, Inductor_SMD:L_Vishay_IHLP-1616, symbol Device:L
- added C1, C2: 1uF, Capacitor_SMD:C_0805_2012Metric_Pad1.18x1.45mm_HandSolder, symbol Device:C
- added C13, C14, C15, C16, C17, C18, C19, C20, C3, C4: 100nF, Capacitor_SMD:C_0805_2012Metric_Pad1.18x1.45mm_HandSolder, symbol Device:C
- added C5, C6, C7, C8: 10uF, Capacitor_SMD:C_0805_2012Metric_Pad1.18x1.45mm_HandSolder, symbol Device:C
- added D1, D3, D5: LED_5V, Diode_SMD:D_0805_2012Metric_Pad1.15x1.40mm_HandSolder, symbol Device:LED
- added D2, D6: D_Schottky, Diode_SMD:D_0805_2012Metric_Pad1.15x1.40mm_HandSolder, symbol Device:D_Schottky
- added D4, D7: 1N4148, Diode_SMD:D_0805_2012Metric_Pad1.15x1.40mm_HandSolder, symbol Diode:1N4148
- added J1: Conn_01x26_Male, Konektor:64734231, symbol Connector:Conn_01x26_Male
- added J2: Conn_02x05_Odd_Even, Connector_PinHeader_2.54mm:PinHeader_2x05_P2.54mm_Vertical, symbol Connector_Generic:Conn_02x05_Odd_Even
- added L1, L2: 10uH, Inductor_SMD:L_Vishay_IHLP-1616, symbol Device:L
- added PS1, PS2: MP2359DT-LF-P, Package_SO:SOIC-8-1EP_3.9x4.9mm_P1.27mm_EP2.29x3mm_ThermalVias, symbol MP2359DT-LF-P:MP2359DT-LF-P
- added R1: R_Small, Resistor_SMD:R_0805_2012Metric_Pad1.20x1.40mm_HandSolder, symbol Device:R_Small
- added R2, R3: 100k, Resistor_SMD:R_0805_2012Metric_Pad1.20x1.40mm_HandSolder, symbol Device:R
- added Y1: Crystal_GND24_Small, Crystal:Crystal_SMD_3225-4Pin_3.2x2.5mm_HandSoldering, symbol Device:Crystal_GND24_Small
- C12: renamed from C?; footprint (none) -> Capacitor_SMD:C_0805_2012Metric_Pad1.18x1.45mm_HandSolder
- FB1: renamed from FB?; footprint (none) -> Capacitor_SMD:C_1812_4532Metric_Pad1.57x3.40mm_HandSolder
- H1, H2, H3, H4: renamed from H?; footprint (none) -> MountingHole:MountingHole_5mm_Pad_Via
- JP1: renamed from JP?; footprint (none) -> Jumper:SolderJumper-3_P1.3mm_Open_RoundedPad1.0x1.5mm
- JP2: renamed from JP?; footprint (none) -> Jumper:SolderJumper-2_P1.3mm_Open_Pad1.0x1.5mm
- R4: renamed from R?; footprint (none) -> Resistor_SMD:R_0805_2012Metric_Pad1.20x1.40mm_HandSolder
- gave numbers to parts that had none: 2
Connections:
- net labels added: +3.3VA, LED_STATUS, NRST, SWCLK, SWDIO, SWO, VSS_IN_1, VSS_IN_2
- net labels removed: +12L
- wire segments 50 -> 163
Other:
- moved on the sheet: C12, FB1, U1

Commit message: almost finished - space for Bartek
Changed lines of the file:
@@
 L power:+5V #PWR0125
 U 1 1 62414F00
-P 1350 5100
-F 0 "#PWR0125" H 1350 4950 50  0001 C CNN
-F 1 "+5V" V 1365 5228 50  0000 L CNN
-F 2 "" H 1350 5100 50  0001 C CNN
-F 3 "" H 1350 5100 50  0001 C CNN
-	1    1350 5100
+P 1350 5500
+F 0 "#PWR0125" H 1350 5350 50  0001 C CNN
+F 1 "+5V" V 1365 5628 50  0000 L CNN
+F 2 "" H 1350 5500 50  0001 C CNN
+F 3 "" H 1350 5500 50  0001 C CNN
+	1    1350 5500
 	0    1    1    0
 $EndComp
@@
 	7600 4400 7600 4550
 $Comp
-L power:+3.3V #PWR0116
-U 1 1 627F0F17
-P 9000 3950
-F 0 "#PWR0116" H 9000 3800 50  0001 C CNN
-F 1 "+3.3V" H 9015 4123 50  0000 C CNN
-F 2 "" H 9000 3950 50  0001 C CNN
-F 3 "" H 9000 3950 50  0001 C CNN
-	1    9000 3950
-	1    0    0    -1
-$EndComp
-$Comp
 L power:GND #PWR0117
 U 1 1 627F0F1D
@@
 	10950 3450 11100 3450
 Connection ~ 11100 3150
+$Comp
+L power:+5V #PWR0116
+U 1 1 629909F8
+P 9000 3950
+F 0 "#PWR0116" H 9000 3800 50  0001 C CNN
+F 1 "+5V" H 9015 4123 50  0000 C CNN
+F 2 "" H 9000 3950 50  0001 C CNN
+F 3 "" H 9000 3950 50  0001 C CNN
+	1    9000 3950
+	1    0    0    -1
+$EndComp
 $EndSCHEMATC

Commit message: Telemetry back v1.0 (#27)
* init commit

* New brd design & final scheme

* final scheme & 60%pcb

* almost finished - space for Bartek

* pre_finnal

* pre_finnal

* telemetry_back_finnal

* Telemetry_back_finnal

* kicad libs

* Create _autosave-telemetria tyl.sch

* Telemetry_back_finnal

* finnal

* Remove Dashboard files from this branch

This reverts commit ffcd00ee911598f18239aabaf1713ea3aea0f91a.

Co-authored-by: wojtekszamocki <w.szamocki.02@gmail.com>
Co-authored-by: Bartosz Janicki <janicki.bartosz.0@gmail.com>
Parts:
- removed JP1: Jumper_3_Bridged12, Jumper:SolderJumper-3_P1.3mm_Open_RoundedPad1.0x1.5mm, symbol Jumper:Jumper_3_Bridged12
- removed JP2: Jumper, Jumper:SolderJumper-2_P1.3mm_Open_Pad1.0x1.5mm, symbol Device:Jumper
- added 2channel_pot1: MAX5478EUD+T, SamacSys_Parts:SOP65P640X110-14N, symbol MAX5478EUD+T:MAX5478EUD+T
- added BJT1: BC846BW,115, SamacSys_Parts:SOT65P210X110-3N, symbol BC846BW:BC846BW
- added C10, C11, C21, C22: C, Capacitor_SMD:C_0805_2012Metric_Pad1.18x1.45mm_HandSolder, symbol Device:C
- added C23: ?, Capacitor_SMD:C_0805_2012Metric_Pad1.18x1.45mm_HandSolder, symbol Device:C
- added C24: 10uF, Capacitor_SMD:C_0805_2012Metric_Pad1.18x1.45mm_HandSolder, symbol Device:C
- added C9: 0.1uF, Capacitor_SMD:C_0805_2012Metric_Pad1.18x1.45mm_HandSolder, symbol Device:C
- added IC1, IC2, IC3: LM741CN_NOPB, DIP794W53P254L959H508Q8N, symbol LM741CN_NOPB:LM741CN_NOPB
- added IC4: NCX2200GW,125, SamacSys_Parts:NCX2200GW, symbol NCX2200GW_125:NCX2200GW,125
- added Mini_DIN_IN1: 5749268-1, SamacSys_Parts:57492681, symbol 5749268-1:5749268-1
- added Mini_DIN_OUT1: 5750071-1, SamacSys_Parts:57500711, symbol 5750071-1:5750071-1
- added Q1: PMV280ENEAR, SamacSys_Parts:PMV280ENEAR, symbol PMV280ENEAR:PMV280ENEAR
- added R10, R14, R15, R16, R17, R18, R23: R, Resistor_SMD:R_0805_2012Metric_Pad1.20x1.40mm_HandSolder, symbol Device:R
- added R19: R?, Resistor_SMD:R_0805_2012Metric_Pad1.20x1.40mm_HandSolder, symbol Device:R
- added R20: 3.3k, Resistor_SMD:R_0805_2012Metric_Pad1.20x1.40mm_HandSolder, symbol Device:R
- added R21: 4.7k, Resistor_SMD:R_0805_2012Metric_Pad1.20x1.40mm_HandSolder, symbol Device:R
- added R22: 1k, Resistor_SMD:R_0805_2012Metric_Pad1.20x1.40mm_HandSolder, symbol Device:R
- added R9: 1M, Resistor_SMD:R_0805_2012Metric_Pad1.20x1.40mm_HandSolder, symbol Device:R
- added RV1: R_POT, Potentiometer_THT:Potentiometer_Alps_RK09L_Single_Vertical, symbol Device:R_POT
- PS1, PS2: footprint Package_SO:SOIC-8-1EP_3.9x4.9mm_P1.27mm_EP2.29x3mm_ThermalVias -> SamacSys_Parts:SOT95P280X145-6N; symbol MP2359DT-LF-P:MP2359DT-LF-P -> telemetria-tyl-rescue:MP2359DT-LF-P-MP2359DT-LF-P
- R4: value R -> 120
Connections:
- net labels added: ADC1_IN0_AMORKI, ADC2_IN1_AMORKI, BREAK_PRESSURE_0, BREAK_PRESSURE_ADC, GND_MIC&ANC, GND_SPK, LED_GND, PTT, SPK+, TX_DATA, V_ANC, V_MIC, V_OUT
- net labels removed: ADC1_IN0, ADC2_IN1
- wire segments 163 -> 214
- no-connect marks 0 -> 26
Other:
- note added: "DIN_IN\n"
- note added: "DIN_OUT\n"
- note added: "PUSH TO TALK \n"
- moved on the sheet: 0.33k1, 0.33k2, 10k1, 10nF1, 1k1, 1k2, 1uF1, 2.2uF1, 2.2uF2, 39nH1, C1, C12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

Commit message: Telemetry_back v1.1 (#31)
* Telemetry_back v1.1

* Telemetry_back_v1.1

* Telemetry_back_v1.1
Parts:
- 10nF1, 1uF1, C12, C13, C14, C15, C16, C17, C18, C19, C20, C3, C4, C5, C6, C7, C8, C9: symbol Device:C -> telemetria-tyl-rescue:C-Device-telemetria-tyl-rescue-telemetria-tyl-rescue
- 2.2uF1, 2.2uF2: symbol Device:C_Small -> telemetria-tyl-rescue:C_Small-Device-telemetria-tyl-rescue-telemetria-tyl-rescue
- 2channel_pot1: symbol MAX5478EUD+T:MAX5478EUD+T -> telemetria-tyl-rescue:MAX5478EUD+T-MAX5478EUD+T-telemetria-tyl-rescue-telemetria-tyl-rescue
- 39nH1, L1, L2: symbol Device:L -> telemetria-tyl-rescue:L-Device-telemetria-tyl-rescue-telemetria-tyl-rescue
- BJT1: symbol BC846BW:BC846BW -> telemetria-tyl-rescue:BC846BW-BC846BW-telemetria-tyl-rescue-telemetria-tyl-rescue
- C1, C2: value 1uF -> 14pF; symbol Device:C -> telemetria-tyl-rescue:C-Device-telemetria-tyl-rescue-telemetria-tyl-rescue
- C10: value C -> 1u; symbol Device:C -> telemetria-tyl-rescue:C-Device-telemetria-tyl-rescue-telemetria-tyl-rescue
- C11, C21: value C -> 1n; symbol Device:C -> telemetria-tyl-rescue:C-Device-telemetria-tyl-rescue-telemetria-tyl-rescue
- C22: value C -> 10n; symbol Device:C -> telemetria-tyl-rescue:C-Device-telemetria-tyl-rescue-telemetria-tyl-rescue
- C23: value ? -> 1uF; symbol Device:C -> telemetria-tyl-rescue:C-Device-telemetria-tyl-rescue-telemetria-tyl-rescue
- C24: value 10uF -> 1uF; symbol Device:C -> telemetria-tyl-rescue:C-Device-telemetria-tyl-rescue-telemetria-tyl-rescue
- D1, D3, D5: value LED_5V -> LED_3.2V; symbol Device:LED -> telemetria-tyl-rescue:LED-Device-telemetria-tyl-rescue-telemetria-tyl-rescue
- D2, D6: symbol Device:D_Schottky -> telemetria-tyl-rescue:D_Schottky-Device-telemetria-tyl-rescue-telemetria-tyl-rescue
- D4, D7: footprint Diode_SMD:D_0805_2012Metric_Pad1.15x1.40mm_HandSolder -> Diode_SMD:D_SOD-123F; symbol Diode:1N4148 -> telemetria-tyl-rescue:1N4148-Diode-telemetria-tyl-rescue-telemetria-tyl-rescue
- FB1: symbol Device:Ferrite_Bead -> telemetria-tyl-rescue:Ferrite_Bead-Device-telemetria-tyl-rescue-telemetria-tyl-rescue
- H1, H2, H3, H4: symbol Mechanical:MountingHole_Pad -> telemetria-tyl-rescue:MountingHole_Pad-Mechanical-telemetria-tyl-rescue-telemetria-tyl-rescue
- IC1, IC2, IC3: symbol LM741CN_NOPB:LM741CN_NOPB -> telemetria-tyl-rescue:LM741CN_NOPB-LM741CN_NOPB-telemetria-tyl-rescue-telemetria-tyl-rescue
- IC4: symbol NCX2200GW_125:NCX2200GW,125 -> telemetria-tyl-rescue:NCX2200GW,125-NCX2200GW_125-telemetria-tyl-rescue-telemetria-tyl-rescue
- J1: symbol Connector:Conn_01x26_Male -> telemetria-tyl-rescue:Conn_01x26_Male-Connector-telemetria-tyl-rescue-telemetria-tyl-rescue
- J2: symbol Connector_Generic:Conn_02x05_Odd_Even -> telemetria-tyl-rescue:Conn_02x05_Odd_Even-Connector_Generic-telemetria-tyl-rescue-telemetria-tyl-rescue
- Mini_DIN_IN1: symbol 5749268-1:5749268-1 -> telemetria-tyl-rescue:5749268-1-5749268-1-telemetria-tyl-rescue-telemetria-tyl-rescue
- Mini_DIN_OUT1: symbol 5750071-1:5750071-1 -> telemetria-tyl-rescue:5750071-1-5750071-1-telemetria-tyl-rescue-telemetria-tyl-rescue
- PS1, PS2: symbol telemetria-tyl-rescue:MP2359DT-LF-P-MP2359DT-LF-P -> telemetria-tyl-rescue:MP2359DT-LF-P-MP2359DT-LF-P-telemetria-tyl-rescue-telemetria-tyl-rescue-telemetria-tyl-rescue
- Q1: symbol PMV280ENEAR:PMV280ENEAR -> telemetria-tyl-rescue:PMV280ENEAR-PMV280ENEAR-telemetria-tyl-rescue-telemetria-tyl-rescue
- R: renamed from 1k1; value R -> 1k; symbol Device:R -> telemetria-tyl-rescue:R-Device-telemetria-tyl-rescue-telemetria-tyl-rescue
- R1: symbol Device:R_Small -> telemetria-tyl-rescue:R_Small-Device-telemetria-tyl-rescue-telemetria-tyl-rescue
- R10: value R -> 1k; symbol Device:R -> telemetria-tyl-rescue:R-Device-telemetria-tyl-rescue-telemetria-tyl-rescue
- R11: value R -> 560; symbol Device:R -> telemetria-tyl-rescue:R-Device-telemetria-tyl-rescue-telemetria-tyl-rescue
- R12, R13: value R -> 360; symbol Device:R -> telemetria-tyl-rescue:R-Device-telemetria-tyl-rescue-telemetria-tyl-rescue
- R14: value R -> 22k; symbol Device:R -> telemetria-tyl-rescue:R-Device-telemetria-tyl-rescue-telemetria-tyl-rescue
- R15, R17: value R -> 10k; symbol Device:R -> telemetria-tyl-rescue:R-Device-telemetria-tyl-rescue-telemetria-tyl-rescue
- R16: value R -> 13k; symbol Device:R -> telemetria-tyl-rescue:R-Device-telemetria-tyl-rescue-telemetria-tyl-rescue
- R18: value R -> 3k; symbol Device:R -> telemetria-tyl-rescue:R-Device-telemetria-tyl-rescue-telemetria-tyl-rescue
- R19: value R? -> 3k; symbol Device:R -> telemetria-tyl-rescue:R-Device-telemetria-tyl-rescue-telemetria-tyl-rescue
- R2, R20, R21, R22, R3, R4, R9: symbol Device:R -> telemetria-tyl-rescue:R-Device-telemetria-tyl-rescue-telemetria-tyl-rescue
- R23: value R -> 4.7k; symbol Device:R -> telemetria-tyl-rescue:R-Device-telemetria-tyl-rescue-telemetria-tyl-rescue
- R5: value R -> 510; symbol Device:R -> telemetria-tyl-rescue:R-Device-telemetria-tyl-rescue-telemetria-tyl-rescue
- R6, R8: value R -> 2k7; symbol Device:R -> telemetria-tyl-rescue:R-Device-telemetria-tyl-rescue-telemetria-tyl-rescue
- R7: value R -> 820; symbol Device:R -> telemetria-tyl-rescue:R-Device-telemetria-tyl-rescue-telemetria-tyl-rescue
- R?: renamed from 0.33k1; value R -> 330; symbol Device:R -> telemetria-tyl-rescue:R-Device-telemetria-tyl-rescue-telemetria-tyl-rescue
- R?: renamed from 1k2; value R -> 1k; symbol Device:R -> telemetria-tyl-rescue:R-Device-telemetria-tyl-rescue-telemetria-tyl-rescue
- R?: renamed from 0.33k2; value R -> 330; symbol Device:R -> telemetria-tyl-rescue:R-Device-telemetria-tyl-rescue-telemetria-tyl-rescue
- R?: renamed from 10k1; value R -> 10k; symbol Device:R -> telemetria-tyl-rescue:R-Device-telemetria-tyl-rescue-telemetria-tyl-rescue
- RV1: symbol Device:R_POT -> telemetria-tyl-rescue:R_POT-Device-telemetria-tyl-rescue-telemetria-tyl-rescue
- U1: symbol MCU_ST_STM32F4:STM32F405RGTx -> telemetria-tyl-rescue:STM32F405RGTx-MCU_ST_STM32F4-telemetria-tyl-rescue-telemetria-tyl-rescue
- U2: symbol Interface_CAN_LIN:MCP2561-E-SN -> telemetria-tyl-rescue:MCP2561-E-SN-Interface_CAN_LIN-telemetria-tyl-rescue-telemetria-tyl-rescue
- Y1: value Crystal_GND24_Small -> 16Mhz; symbol Device:Crystal_GND24_Small -> telemetria-tyl-rescue:Crystal_GND24_Small-Device-telemetria-tyl-rescue-telemetria-tyl-rescue
