File: BSPD/BSPD.kicad_pcb (KiCad board)
At the start: 2 copper layers, 52.1 x 29.2 mm, 47 parts, among them IC1 SN74AHC1G02DBVR, IC2 LM393AD, IC3 LM393AD, IC4 LM393AD, J1 Conn_02x03_Odd_Even, K1 CP1-12V, Q1 Si2319CDS, Q2 BSS138, Q3 BSS138, U1 LM1117-5.0

Commit message: BSPD
With Gerbers
Parts:
- added D3: 1N4148W, Diode_SMD:D_SOD-123, B.Cu at (139.7, 90.2)
- added H1: MountingHole_Pad, MountingHole:MountingHole_2.2mm_M2_Pad_Via, F.Cu at (111.8, 76.2)
- added H2: MountingHole_Pad, MountingHole:MountingHole_2.2mm_M2_Pad_Via, F.Cu at (143.5, 76.2)
- added H3: MountingHole_Pad, MountingHole:MountingHole_2.2mm_M2_Pad_Via, F.Cu at (143.5, 101.6)
- added H4: MountingHole_Pad, MountingHole:MountingHole_2.2mm_M2_Pad_Via, F.Cu at (111.8, 101.6)
- moved RV1 0.15 mm to (99.2, 91.5)
- moved RV2 0.15 mm to (105.6, 91.5)
Connections:
- RV1 pad 1: +5V -> Net-(RV1-Pad1)
- RV1 pad 2: Net-(IC2-Pad3) -> +5V
- RV1 pad 3: GND -> Net-(IC2-Pad3)
- RV2 pad 1: +5V -> Net-(RV2-Pad1)
- RV2 pad 2: Net-(IC3-Pad3) -> +5V
- RV2 pad 3: GND -> Net-(IC3-Pad3)
Routing:
- net GND: track 183.2 -> 223.6 mm
- net TRIG: track 57.5 -> 69.8 mm
- net +12V: track 44.2 -> 49.2 mm
- net Net-(IC2-Pad3): track 17.6 -> 19.4 mm
- net Net-(D3-Pad2): track 14.5 -> 16.2 mm
- net Net-(IC3-Pad3): track 23.5 -> 24.5 mm
- net COMP2: track 27.3 -> 28.0 mm
- net +5V: track 162.2 -> 162.1 mm, vias 4 -> 3
Other:
- board size 52.1 x 29.2 mm -> 52.1 x 31.8 mm
- board text added: "BSPD by Janicki"
