File: BSPD/BSPD.sch (KiCad schematic (older format))
At the start: 47 parts, among them IC1 SN74AHC1G02DBVR, IC2 LM393AD, IC3 LM393AD, IC4 LM393AD, J1 Conn_02x03_Odd_Even, K1 CP1-12V, Q1 Si2319CDS, Q2 BSS138, Q3 BSS138, U1 LM1117-5.0

Commit message: BSPD
With Gerbers
Parts:
- added D3: 1N4148W, Diode_SMD:D_SOD-123, symbol BSPD-rescue:1N4148W-Diode
- added H1, H2, H3, H4: MountingHole_Pad, MountingHole:MountingHole_2.2mm_M2_Pad_Via, symbol BSPD-rescue:MountingHole_Pad-Mechanical
- C1, C10, C2, C3, C4, C5, C6, C7, C8, C9: symbol Device:C -> BSPD-rescue:C-Device
- J1: symbol Connector_Generic:Conn_02x03_Odd_Even -> BSPD-rescue:Conn_02x03_Odd_Even-Connector_Generic
- Q1: symbol Transistor_FET:Si2319CDS -> BSPD-rescue:Si2319CDS-Transistor_FET
- Q2, Q3: symbol Transistor_FET:BSS138 -> BSPD-rescue:BSS138-Transistor_FET
- R1, R10, R11, R12, R13, R14, R15, R16, R17, R18, R19, R2, R20, R21, R22, R23, R24, R25, R3, R4, R6, R8, R9: symbol Device:R -> BSPD-rescue:R-Device
- RV1, RV2: symbol Device:R_POT -> BSPD-rescue:R_POT-Device
- U1: symbol Regulator_Linear:LM1117-5.0 -> BSPD-rescue:LM1117-5.0-Regulator_Linear
Connections:
- net +12V: now also D3.1 (K)
- net +5V: now also RV1.2, RV2.2; no longer RV1.1, RV2.1
- net GND: now also H1.1, H2.1, H3.1, H4.1; no longer RV1.3, RV2.3
- net at IC2.3 (1IN+), R6.2: now also RV1.3; no longer RV1.2
- net at IC3.3 (1IN+), R8.2: now also RV2.3; no longer RV2.2
- net at K1.5 (COIL_2), Q2.3 (D): now also D3.2 (A)
- no-connect marks 0 -> 1
Other:
- moved on the sheet: RV1, RV2
