File: CAN2USB/PCB/can2usb/can2usb.kicad_pcb (KiCad board)
At the start: 2 copper layers, 32 parts, among them SW2 RESET_SW, U1 STM32F103C6Tx, U2 TLP175A, U3 MCP2561-E-SN, U4 LM1117-3.3

Commit message: Minor changes, attached footprints
Parts:
- removed C11: 100nF, Capacitor_SMD:C_0805_2012Metric
- removed R9: 10k, Resistor_SMD:R_0805_2012Metric
- removed SW2: RESET_SW, Button_Switch_SMD:SW_Push_1P1T_NO_CK_KMR2
- added J1: STLINK, Connector_PinHeader_2.54mm:PinHeader_1x04_P2.54mm_Vertical, F.Cu at (49.5, 25.4)
- added J2: Conn_01x03_Male, Connector_PinHeader_2.54mm:PinHeader_1x03_P2.54mm_Vertical, F.Cu at (58.4, 17.8)
- added P1: USB_C_Plug_USB2.0, Connector_USB:USB_C_Receptacle_GCT_USB4085, F.Cu at (54.7, 24.7)
- added SW1: BOOT_SW, Button_Switch_SMD:SW_SPDT_PCM12, F.Cu at (51.2, 18.4)
- added Y1: 16MHz, Crystal:Crystal_SMD_5032-2Pin_5.0x3.2mm, F.Cu at (49.9, 24.8)
- added Y2: 32KHz, Crystal:Crystal_SMD_3215-2Pin_3.2x1.5mm, F.Cu at (63.3, 17.1)
- moved D2 24.8 mm to (44.4, 16.9)
- moved R2 24.7 mm to (29.4, 34.5)
- moved C9 22.7 mm to (39.4, 19.9)
- moved D1 21.2 mm to (29.4, 31.5)
- moved F1 18.2 mm to (43.8, 19.9)
- moved C5 17.3 mm to (25.0, 31.4)
- moved C3 17.2 mm to (25.0, 28.4)
- moved C10 17.1 mm to (25.0, 34.5)
- moved C6 15.2 mm to (40.0, 16.8)
- moved R8 15.0 mm to (43.8, 25.8)
- moved C4 14.7 mm to (34.9, 22.0)
- moved C2 13.5 mm to (35.5, 16.8)
- moved R7 13.0 mm to (38.3, 28.8)
- moved R_CONF2 13.0 mm to (42.7, 28.8)
- moved R4 12.8 mm to (33.9, 31.4)
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Connections:
- F1 pad 1: (no net) -> Net-(F1-Pad1)
- R1 pad 1: (no net) -> Net-(P1-PadA5)
- R8 pad 2: (no net) -> Net-(R8-Pad2)
- U1 pad 1: (no net) -> +3V3
- U1 pad 34: (no net) -> SWDIO
- U1 pad 37: (no net) -> SWCLK
- U1 pad 7: NRST -> (no net)
