File: CAN2USB/PCB/can2usb/can2usb.sch (KiCad schematic (older format))
At the start: 29 parts, among them P1 USB_C_Plug_USB2.0, U1 STM32F103C6Tx, U2 TLP175A, U3 MCP2561-E-SN, Y1 16MHz, Y2 32KHz

Commit message: Final schematic
Parts:
- added C10, C9: 10uF, Capacitor_SMD:C_0805_2012Metric, symbol Device:C_Small
- added C11: 100nF, Capacitor_SMD:C_0805_2012Metric, symbol Device:C_Small
- added R8: 1k, Resistor_SMD:R_0805_2012Metric, symbol Device:R_Small
- added R9: 10k, Resistor_SMD:R_0805_2012Metric, symbol Device:R_Small
- added SW1: BOOT_SW, symbol Switch:SW_SPDT
- added SW2: RESET_SW, Button_Switch_SMD:SW_Push_1P1T_NO_CK_KMR2, symbol Switch:SW_Push
- C1, C2, C3, C4, C5, C6, C7, C8: footprint (none) -> Capacitor_SMD:C_0805_2012Metric
- D1, D2, D3: footprint (none) -> LED_SMD:LED_0805_2012Metric
- F1: footprint (none) -> Fuse:Fuse_0805_2012Metric
- R1, R2, R3, R4, R5, R6, R7, R_CONF1, R_CONF2, R_Terminator1: footprint (none) -> Resistor_SMD:R_0805_2012Metric
- U4: renamed from U?; footprint (none) -> Package_TO_SOT_SMD:SOT-223-3_TabPin2
Connections:
- net +3V3: now also U4.2 (VO), C10.2, R9.1, SW1.3 (C)
- net +5V: now also U4.3 (VI), C9.2
- net GND: now also C10.1, C11.2, C9.1, SW1.1 (A), SW2.1
- net BOOT0: now reaches U1.44 (BOOT0)
- net BOOT0: now also R8.1
- net NRST: now reaches U1.7 (NRST)
- net NRST: now also C11.1, R9.2, SW2.2
- new net: R8.2, SW1.2 (B)
- no-connect marks 2 -> 28
Other:
- note added: "LDO\n"
- moved on the sheet: C1, C2, C3, C4, U1, U4

Commit message: Minor changes, attached footprints
Parts:
- removed C11: 100nF, Capacitor_SMD:C_0805_2012Metric, symbol Device:C_Small
- removed R9: 10k, Resistor_SMD:R_0805_2012Metric, symbol Device:R_Small
- removed SW2: RESET_SW, Button_Switch_SMD:SW_Push_1P1T_NO_CK_KMR2, symbol Switch:SW_Push
- added J1: STLINK, Connector_PinHeader_2.54mm:PinHeader_1x04_P2.54mm_Vertical, symbol Connector:Conn_01x04_Male
- added J2: Conn_01x03_Male, Connector_PinHeader_2.54mm:PinHeader_1x03_P2.54mm_Vertical, symbol Connector:Conn_01x03_Male
- P1: footprint (none) -> Connector_USB:USB_C_Receptacle_GCT_USB4085
- SW1: footprint (none) -> Button_Switch_SMD:SW_SPDT_PCM12
- Y1: footprint (none) -> Crystal:Crystal_SMD_5032-2Pin_5.0x3.2mm
- Y2: footprint (none) -> Crystal:Crystal_SMD_3215-2Pin_3.2x1.5mm
Connections:
- net +3V3: now also U1.1 (VBAT)
- net +5V: now also J1.1 (Pin_1)
- net CAN_H: now also J2.2 (Pin_2)
- net CAN_L: now also J2.1 (Pin_1)
- net GND: now also J1.4 (Pin_4), J2.3 (Pin_3); no longer P1.S1 (SHIELD)
- net SWDIO: now reaches U1.34 (PA13)
- net SWDIO: now also J1.3 (Pin_3)
- net SWCLK: now reaches U1.37 (PA14)
- net SWCLK: now also J1.2 (Pin_2)
- net NRST: no longer names the net of U1.7 (NRST)
- no-connect marks 28 -> 27
Changed lines of the file:
@@
 F 0 "P1" H 9732 2542 50  0000 C CNN
 F 1 "USB_C_Plug_USB2.0" H 9732 2451 50  0000 C CNN
-F 2 "" H 9775 1675 50  0001 C CNN
+F 2 "Connector_USB:USB_C_Receptacle_GCT_USB4085" H 9775 1675 50  0001 C CNN
 F 3 "https://www.usb.org/sites/default/files/documents/usb_type-c.zip" H 9775 1675 50  0001 C CNN
 	1    9625 1675
@@
 L power:GND #PWR0109
 U 1 1 63311987
-P 9475 2625
-F 0 "#PWR0109" H 9475 2375 50  0001 C CNN
-F 1 "GND" H 9480 2452 50  0000 C CNN
-F 2 "" H 9475 2625 50  0001 C CNN
-F 3 "" H 9475 2625 50  0001 C CNN
-	1    9475 2625
-	1    0    0    -1
-$EndComp
-Wire Wire Line
-	9325 2575 9325 2625
-Wire Wire Line
-	9325 2625 9475 2625
-Wire Wire Line
-	9475 2625 9625 2625
-Connection ~ 9475 2625
+P 9625 2625
+F 0 "#PWR0109" H 9625 2375 50  0001 C CNN
+F 1 "GND" H 9630 2452 50  0000 C CNN
+F 2 "" H 9625 2625 50  0001 C CNN
+F 3 "" H 9625 2625 50  0001 C CNN
+	1    9625 2625
+	1    0    0    -1
+$EndComp
 NoConn ~ 10225 1375
 Text GLabel 1550 3575 0    50   Input ~ 0
@@
 F 0 "Y1" H 7975 2050 50  0000 C CNN
 F 1 "16MHz" H 7975 1959 50  0000 C CNN
-F 2 "" H 7975 1825 50  0001 C CNN
+F 2 "Crystal:Crystal_SMD_5032-2Pin_5.0x3.2mm" H 7975 1825 50  0001 C CNN
 F 3 "~" H 7975 1825 50  0001 C CNN
 	1    7975 1825
@@
 F 0 "Y2" H 6500 1950 50  0000 C CNN
 F 1 "32KHz" H 6500 1859 50  0000 C CNN
-F 2 "" H 6500 1725 50  0001 C CNN
+F 2 "Crystal:Crystal_SMD_3215-2Pin_3.2x1.5mm" H 6500 1725 50  0001 C CNN
 F 3 "~" H 6500 1725 50  0001 C CNN
 	1    6500 1725
@@
 F 0 "SW1" H 1300 5600 50  0000 C CNN
 F 1 "BOOT_SW" H 1300 5691 50  0000 C CNN
-F 2 "" H 1300 5925 50  0001 C CNN
+F 2 "Button_Switch_SMD:SW_SPDT_PCM12" H 1300 5925 50  0001 C CNN
 F 3 "~" H 1300 5925 50  0001 C CNN
 	1    1300 5925
@@
 Text GLabel 1475 1875 0    50   Input ~ 0
 BOOT0
-Text GLabel 1550 1675 0    50   Input ~ 0
-NRST
 Text GLabel 1750 5925 2    50   Input ~ 0
 BOOT0
-Wire Wire Line
-	1425 7325 1425 7175
-$Comp
-L power:GND #PWR018
-U 1 1 6333EB03
-P 1425 7325
-F 0 "#PWR018" H 1425 7075 50  0001 C CNN
-F 1 "GND" H 1430 7152 50  0000 C CNN
-F 2 "" H 1425 7325 50  0001 C CNN
-F 3 "" H 1425 7325 50  0001 C CNN
-	1    1425 7325
-	1    0    0    -1
-$EndComp
-Wire Wire Line
-	1425 6900 1450 6900
-Connection ~ 1425 6900
-Wire Wire Line
-	1425 6900 1425 6975
-$Comp
-L Device:C_Small C11
-U 1 1 6333C1F1
-P 1425 7075
-F 0 "C11" H 1517 7121 50  0000 L CNN
-F 1 "100nF" H 1517 7030 50  0000 L CNN
-F 2 "Capacitor_SMD:C_0805_2012Metric" H 1425 7075 50  0001 C CNN
-F 3 "~" H 1425 7075 50  0001 C CNN
-	1    1425 7075
-	1    0    0    -1
-$EndComp
-Wire Wire Line
-	925  6575 925  6475
-$Comp
-L power:+3.3V #PWR016
-U 1 1 6333874E
-P 925 6475
-F 0 "#PWR016" H 925 6325 50  0001 C CNN
-F 1 "+3.3V" H 940 6648 50  0000 C CNN
-F 2 "" H 925 6475 50  0001 C CNN
-F 3 "" H 925 6475 50  0001 C CNN
-	1    925  6475
-	1    0    0    -1
-$EndComp
-Connection ~ 925  6900
-Wire Wire Line
-	925  6900 925  6775
-$Comp
-L Device:R_Small R9
-U 1 1 6333601B
-P 925 6675
-F 0 "R9" H 984 6721 50  0000 L CNN
-F 1 "10k" H 984 6630 50  0000 L CNN
-F 2 "Resistor_SMD:R_0805_2012Metric" H 925 6675 50  0001 C CNN
-F 3 "~" H 925 6675 50  0001 C CNN
-	1    925  6675
-	1    0    0    -1
-$EndComp
-Wire Wire Line
-	925  6900 1425 6900
-Text GLabel 1450 6900 2    50   Input ~ 0
-NRST
-$Comp
-L power:GND #PWR017
-U 1 1 6332CD7C
-P 925 7300
-F 0 "#PWR017" H 925 7050 50  0001 C CNN
-F 1 "GND" H 930 7127 50  0000 C CNN
-F 2 "" H 925 7300 50  0001 C CNN
-F 3 "" H 925 7300 50  0001 C CNN
-	1    925  7300
-	1    0    0    -1
-$EndComp
-$Comp
-L Switch:SW_Push SW2
-U 1 1 6331845C
-P 925 7100
-F 0 "SW2" V 971 7052 50  0000 R CNN
-F 1 "RESET_SW" V 880 7052 50  0000 R CNN
-F 2 "Button_Switch_SMD:SW_Push_1P1T_NO_CK_KMR2" H 925 7300 50  0001 C CNN
-F 3 "~" H 925 7300 50  0001 C CNN
-	1    925  7100
-	0    -1   -1   0
-$EndComp
 Wire Notes Line
 	4025 475  4025 5525
@@
 NoConn ~ 2850 3675
 NoConn ~ 2850 3775
-NoConn ~ 2850 4075
-NoConn ~ 2850 4175
 NoConn ~ 2850 4275
 NoConn ~ 1550 2975
@@
 	1    0    0    -1
 $EndComp
-NoConn ~ 2050 1475
 $Comp
 L power:GND #PWR0101
@@
 Wire Wire Line
 	9625 2575 9625 2625
+$Comp
+L power:PWR_FLAG #FLG0101
+U 1 1 63307A51
+P 9750 2625
+F 0 "#FLG0101" H 9750 2700 50  0001 C CNN
+F 1 "PWR_FLAG" V 9750 2753 50  0000 L CNN
+F 2 "" H 9750 2625 50  0001 C CNN
+F 3 "~" H 9750 2625 50  0001 C CNN
+	1    9750 2625
+	0    1    1    0
+$EndComp
+Wire Wire Line
+	9750 2625 9625 2625
+Text GLabel 2850 4075 2    50   Input ~ 0
+SWDIO
+Text GLabel 2850 4175 2    50   Input ~ 0
+SWCLK
+$Comp
+L Connector:Conn_01x04_Male J1
+U 1 1 6330FED6
+P 3075 6100
+F 0 "J1" H 3047 5982 50  0000 R CNN
+F 1 "STLINK" H 3047 6073 50  0000 R CNN
+F 2 "Connector_PinHeader_2.54mm:PinHeader_1x04_P2.54mm_Vertical" H 3075 6100 50  0001 C CNN
+F 3 "~" H 3075 6100 50  0001 C CNN
+	1    3075 6100
+	-1   0    0    1
+$EndComp
+$Comp
+L power:GND #PWR04
+U 1 1 63316A3C
+P 2675 5900
+F 0 "#PWR04" H 2675 5650 50  0001 C CNN
+F 1 "GND" V 2680 5772 50  0000 R CNN
+F 2 "" H 2675 5900 50  0001 C CNN
+F 3 "" H 2675 5900 50  0001 C CNN
+	1    2675 5900
+	0    1    1    0
+$EndComp
+Wire Wire Line
+	2675 5900 2875 5900
+Text GLabel 2775 6000 0    50   Input ~ 0
+SWDIO
+Wire Wire Line
+	2775 6000 2875 6000
+Text GLabel 2775 6100 0    50   Input ~ 0
+SWCLK
+Wire Wire Line
+	2775 6100 2875 6100
+$Comp
+L power:+5V #PWR012
+U 1 1 63328888
+P 2875 6200
+F 0 "#PWR012" H 2875 6050 50  0001 C CNN
+F 1 "+5V" V 2890 6328 50  0000 L CNN
+F 2 "" H 2875 6200 50  0001 C CNN
+F 3 "" H 2875 6200 50  0001 C CNN
+	1    2875 6200
+	0    -1   -1   0
+$EndComp
+Wire Wire Line
+	2050 1475 2150 1475
+Connection ~ 2150 1475
+Connection ~ 9625 2625
+NoConn ~ 9325 2575
+NoConn ~ 1550 1675
+$Comp
+L power:GND #PWR0115
+U 1 1 63365CEC
+P 2875 6550
+F 0 "#PWR0115" H 2875 6300 50  0001 C CNN
+F 1 "GND" V 2880 6422 50  0000 R CNN
+F 2 "" H 2875 6550 50  0001 C CNN
+F 3 "" H 2875 6550 50  0001 C CNN
+	1    2875 6550
+	0    1    1    0
+$EndComp
+$Comp
+L Connector:Conn_01x03_Male J2
+U 1 1 63366EE1
+P 3075 6650
+F 0 "J2" H 3047 6582 50  0000 R CNN
+F 1 "Conn_01x03_Male" H 3047 6673 50  0000 R CNN
+F 2 "Connector_PinHeader_2.54mm:PinHeader_1x03_P2.54mm_Vertical" H 3075 6650 50  0001 C CNN
+F 3 "~" H 3075 6650 50  0001 C CNN
+	1    3075 6650
+	-1   0    0    1
+$EndComp
+Text GLabel 2875 6650 0    50   Input ~ 0
+CAN_H
+Text GLabel 2875 6750 0    50   Input ~ 0
+CAN_L
 $EndSCHEMATC
