File: GearControl/PCB/GearControl_v3/GearControl.kicad_pcb (KiCad board)
At the start: 4 copper layers, 85.5 x 64 mm, 136 parts, among them IC1 KF50BDT-TR, IC10 KF50BDT-TR, IC2 BTN7970B, IC3 BTN7970B, IC4 74HC126DB,118, IC5 74HC2G16GVH, IC6 NL27WZ14DTT1G, IC7 KF50BDT-TR, IC8 MCP6L02T-E_SN, IC9 MCP6L02T-E_SN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

Commit message: Update GearCtrl PCB for safety system for ETB
Parts:
- added K1: CPC-1017N, CPC-1017N:CPC-1017N, B.Cu at (95.0, 60.0)
- added R59: 10k, Resistor_SMD:R_0603_1608Metric, B.Cu at (94.5, 52.4)
- added R60: 210, Resistor_SMD:R_0603_1608Metric, B.Cu at (96.7, 65.3)
Connections:
- net PWM_CLUTCH_OUT_12V renamed PWM_CLUTCH_OUT_5V
- net PWM_GEAR_OUT_12V renamed PWM_GEAR_OUT_5V
- J1 pad 15: SW_G_DOWN_P2 -> unconnected-(J1-Pad15)
- J1 pad 6: SW_G_DOWN_P2 -> SAFETY_LINE_IN
- J1 pad 7: 5V_APPS -> SAFETY_LINE_OUT
- J1 pad MH1: (no net) -> unconnected-(J1-PadMH1)
- J1 pad MH2: (no net) -> unconnected-(J1-PadMH2)
- U2 pad 11: (no net) -> unconnected-(U2-Pad11)
- U2 pad 14: (no net) -> unconnected-(U2-Pad14)
- U2 pad 2: (no net) -> unconnected-(U2-Pad2)
- U2 pad 20: (no net) -> unconnected-(U2-Pad20)
- U2 pad 22: (no net) -> unconnected-(U2-Pad22)
- U2 pad 24: (no net) -> unconnected-(U2-Pad24)
- U2 pad 26: (no net) -> unconnected-(U2-Pad26)
- U2 pad 28: (no net) -> unconnected-(U2-Pad28)
- U2 pad 29: (no net) -> unconnected-(U2-Pad29)
- U2 pad 3: (no net) -> unconnected-(U2-Pad3)
- U2 pad 30: (no net) -> unconnected-(U2-Pad30)
- U2 pad 33: (no net) -> SAFETY_LINE_CTRL
- U2 pad 34: (no net) -> unconnected-(U2-Pad34)
- U2 pad 36: (no net) -> unconnected-(U2-Pad36)
- U2 pad 38: (no net) -> unconnected-(U2-Pad38)
- U2 pad 4: (no net) -> unconnected-(U2-Pad4)
- U2 pad 45: (no net) -> unconnected-(U2-Pad45)
- U2 pad 50: (no net) -> unconnected-(U2-Pad50)
- U2 pad 51: (no net) -> unconnected-(U2-Pad51)
- U2 pad 52: (no net) -> unconnected-(U2-Pad52)
- U2 pad 53: (no net) -> unconnected-(U2-Pad53)
- U2 pad 54: (no net) -> unconnected-(U2-Pad54)
- U2 pad 56: (no net) -> unconnected-(U2-Pad56)
- U2 pad 57: (no net) -> unconnected-(U2-Pad57)
- U2 pad 58: (no net) -> unconnected-(U2-Pad58)
- U2 pad 59: (no net) -> unconnected-(U2-Pad59)
- U2 pad 8: (no net) -> unconnected-(U2-Pad8)
- U4 pad 5: (no net) -> unconnected-(U4-Pad5)
Routing:
- net SAFETY_LINE_CTRL: track 0.00 -> 90.9 mm, vias 0 -> 4
- net Net-(K1-Pad1): track 0.00 -> 13.6 mm
- net 5V_APPS: track 102.9 -> 92.3 mm
- net SAFETY_LINE_OUT: track 0.00 -> 7.39 mm
- net +3V3: track 119.6 -> 125.2 mm
- net SAFETY_LINE_IN: track 0.00 -> 3.27 mm
Other:
- net class Default removed
